File: pcb/ebc.kicad_pcb (KiCad board)
At the start: 2 copper layers, 90 x 50 mm, 110 parts, among them P1 HE10-10, P2 CONN_01X30, SW1 POWER, U1 M24SR64-Y, U2 MSP432P401R, U3 FAN5331, X1 XC9142

Commit message: - pcb gerbered out and stencils created
Parts:
- added REF**: VIA, rorycad:VIA-0.6MM, F.Cu at (138.6, 95.7)
- added REF**: VIA, rorycad:VIA-0.6MM, F.Cu at (178.3, 110.2)
- added REF**: VIA, rorycad:VIA-0.6MM, F.Cu at (170.4, 111.2)
Connections:
- P2 pad : (no net) -> GND
Routing:
- net GND: track 39.8 -> 57.7 mm, vias 7 -> 11
- net Net-(C13-Pad2): track 7.87 -> 10.2 mm
